File: Zusatzsignal/LED_Matrix_3_1.sch (EAGLE design)
At the start: 61 parts, among them IC1 PIC6C595D, X1 SSW-106-02-S-S

Commit message: Verbesserung der Zusatzanzeigerplatine
- Änderung des Layouts der Rückseite
- Änderung der Durchführungen auf RM
- Beseitigung von DRC-Fehlern
Parts:
- removed S1, S2, S3, S4, S5: (no value), pinhead:PINHD-1X1
- added X2: SSW-102-02-S-S, con-samtec:SSW-102-02-S-S
- added X4: SSW-103-02-S-S, con-samtec:SSW-103-02-S-S
- R1, R10, R11, R12, R16, R5, R6: device eagle-ltspice:RR0603 -> resistor:R-EU_R0603
Connections:
- net N$4: now also R6.2; no longer R5.2
- net N$5: now also R5.2; no longer R6.2
- net S1: now also X4-3.1; no longer S1.1
- net S2: now also X4-2.1; no longer S2.1
- net S3: now also X4-1.1; no longer S3.1
- net S4: now also X2-2.1; no longer S4.1
- net S5: now also X2-1.1; no longer S5.1
